Commit message: altitude pid controls

File: models/drone.urdf (robot description, URDF)
Before this commit: robot drone, 5 links, 4 joints
Links:
- link BL: mass None -> 0.1
- link BR: mass None -> 0.1
- link FL: mass None -> 0.1
- link FR: mass None -> 0.1
- link base_link: mass None -> 0.6
Joints:
- joint base_to_BL: origin (none) -> xyz=0 0 0 rpy=0 0 0
- joint base_to_BR: origin (none) -> xyz=0 0 0 rpy=0 0 0
- joint base_to_FL: origin (none) -> xyz=0 0 0 rpy=0 0 0
- joint base_to_FR: origin (none) -> xyz=0 0 0 rpy=0 0 0
